Commit message: sim für wolfgang weiter anpassen

File: Wolfgang/wolfgang_assets/urdf/robot.urdf (robot description, URDF)
Before this commit: robot wolfgang, 48 links, 47 joints
Links:
- link head: geometry collision box size=0.006 0.072 0.03; collision box size=0.006 0.072 0.03
- link l_ankle: geometry collision box size=0.028 0.0035 0.0059; collision box size=0.028 0.0035 0.0059
- link l_foot: geometry collision box size=0.008 0.04 0.004; collision box size=0.008 0.04 0.004
- link l_hip_1: geometry collision box size=0.0260229 0.004 0.053; collision box size=0.0260229 0.004 0.053
- link l_hip_2: geometry collision box size=0.028 0.0035 0.0059; collision box size=0.028 0.0035 0.0059
- link l_lower_arm: geometry collision box size=0.012 0.002 0.029; collision box size=0.012 0.002 0.029
- link l_lower_leg: geometry collision box size=0.014 0.0091 0.031; collision box size=0.034 0.002 0.16
- link l_shoulder: geometry collision box size=0.0015 0.045 0.028; collision box size=0.0015 0.045 0.028
- link l_upper_arm: geometry collision box size=0.036 0.04 0.0093; collision box size=0.036 0.04 0.0093
- link l_upper_leg: geometry collision box size=0.01 0.002 0.01; collision box size=0.01 0.002 0.01
- link llb: geometry collision cylinder length=0.01 radius=0.006; collision sphere radius=0.006
- link llf: geometry collision cylinder length=0.01 radius=0.006; collision sphere radius=0.006
- link lrb: geometry collision cylinder length=0.01 radius=0.006; collision sphere radius=0.006
- link lrf: geometry collision cylinder length=0.01 radius=0.006; collision sphere radius=0.006
- link neck: geometry collision box size=0.036 0.04 0.0093; collision box size=0.0402 0.041 0.0611
- link r_ankle: geometry collision box size=0.028 0.0035 0.0059; collision box size=0.028 0.0035 0.0059
- link r_foot: geometry collision box size=0.008 0.04 0.004; collision box size=0.008 0.04 0.004
- link r_hip_1: geometry collision box size=0.0260229 0.004 0.053; collision box size=0.0260229 0.004 0.053
- link r_hip_2: geometry collision box size=0.028 0.0035 0.0059; collision box size=0.028 0.0035 0.0059
- link r_lower_arm: geometry collision box size=0.012 0.002 0.029; collision box size=0.012 0.002 0.029
- link r_lower_leg: geometry collision box size=0.014 0.0091 0.031; collision box size=0.034 0.002 0.16
- link r_shoulder: geometry collision box size=0.0015 0.045 0.028; collision box size=0.0015 0.045 0.028
- link r_upper_arm: geometry collision box size=0.036 0.04 0.0093; collision box size=0.036 0.04 0.0093
- link r_upper_leg: geometry collision box size=0.01 0.002 0.01; collision box size=0.01 0.002 0.01
- link rlb: geometry collision cylinder length=0.01 radius=0.006; collision sphere radius=0.006
- link rlf: geometry collision cylinder length=0.01 radius=0.006; collision sphere radius=0.006
- link rrb: geometry collision cylinder length=0.01 radius=0.006; collision sphere radius=0.006
- link rrf: geometry collision cylinder length=0.01 radius=0.006; collision sphere radius=0.006
- link torso: geometry collision box size=0.019 0.0468795 0.005; collision box size=0.019 0.0468795 0.005
